File: Lesson 4/Eagle/DIYpiano/DIYpiano.brd (EAGLE design)
At the start: 110.5 x 43.2 mm, 24 parts, among them IC1 NE555N, Q1 2N2222, SW1 MOMENTARY-SWITCH-SPST-PTH-6.0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, SW2 MOMENTARY-SWITCH-SPST-PTH-6.0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, SW3 MOMENTARY-SWITCH-SPST-PTH-6.0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, SW4 MOMENTARY-SWITCH-SPST-PTH-6.0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, SW5 MOMENTARY-SWITCH-SPST-PTH-6.0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, SW6 MOMENTARY-SWITCH-SPST-PTH-6.0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, SW7 MOMENTARY-SWITCH-SPST-PTH-6.0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, SW8 MOMENTARY-SWITCH-SPST-PTH-6.0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

Commit message: Updates to the BOM/PL of DIY Piano circuit
Parts:
- LS1: value AT-1220-TT-3V-2-R -> (none)
