File: Lesson 4/Eagle/DIYpiano/DIYpiano.sch (EAGLE design)
At the start: 24 parts, among them IC1 NE555N, Q1 2N2222, SW1 MOMENTARY-SWITCH-SPST-PTH-6.0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, SW2 MOMENTARY-SWITCH-SPST-PTH-6.0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, SW3 MOMENTARY-SWITCH-SPST-PTH-6.0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, SW4 MOMENTARY-SWITCH-SPST-PTH-6.0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, SW5 MOMENTARY-SWITCH-SPST-PTH-6.0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, SW6 MOMENTARY-SWITCH-SPST-PTH-6.0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, SW7 MOMENTARY-SWITCH-SPST-PTH-6.0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, SW8 MOMENTARY-SWITCH-SPST-PTH-6.0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

Commit message: Updates to the BOM/PL of DIY Piano circuit
Parts:
- BATT: MOUSER# (none) -> 534-3001
- C1, C2: MOUSER# (none) -> 581-SR201C104KARTR1
- IC1: MOUSER# (none) -> 595-TLC555CP
- LS1: value AT-1220-TT-3V-2-R -> F/HMB; MOUSER# (none) -> 665-AST-01508MR-R
- Q1: MOUSER# (none) -> 833-PN2222A-AP
- R1, R3, R9: MOUSER# (none) -> 660-MF1/4DCT26A1001F
- R10: MOUSER# (none) -> 603-MFR-25FRF52-910R
- R2: MOUSER# (none) -> 603-MFR-25FRF52-6K2
- R4: MOUSER# (none) -> 603-MFR-25FTE52-390R
- R5: MOUSER# (none) -> 603-MFR-25FBF52-1K5
- R6: MOUSER# (none) -> 603-MFR-25FBF52-1K3
- R7: MOUSER# (none) -> 603-MFR-25FBF52-620R
- R8: MOUSER# (none) -> 603-MFR-25FBF52-1K1
- SW1, SW2, SW3, SW4, SW5, SW6, SW7, SW8: MOUSER# (none) -> 653-B3F-1000
