File: Lesson 4/EE-Workshop.sch (EAGLE design)
At the start: 1 part

Commit message: Updates to Lesson 4
Parts:
- BATT: value AB9V -> AB3V
Changed lines of the file:
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@@
 </classes>
 <parts>
-<part name="BATT" library="battery" library_urn="urn:adsk.eagle:library:109" deviceset="AB9V" device="" package3d_urn="urn:adsk.eagle:package:4600/1"/>
+<part name="BATT" library="battery" library_urn="urn:adsk.eagle:library:109" deviceset="AB9V" device="" package3d_urn="urn:adsk.eagle:package:4600/1" value="AB3V"/>
 </parts>
 <sheets>
