File: Lesson 5/E-Piano-SM.sch (EAGLE design)
At the start: 24 parts, among them Q1 BCW66, SW1 MOMENTARY-SWITCH-SPST-SMD-6.2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, SW2 MOMENTARY-SWITCH-SPST-SMD-6.2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, SW3 MOMENTARY-SWITCH-SPST-SMD-6.2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, SW4 MOMENTARY-SWITCH-SPST-SMD-6.2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, SW5 MOMENTARY-SWITCH-SPST-SMD-6.2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, SW6 MOMENTARY-SWITCH-SPST-SMD-6.2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, SW7 MOMENTARY-SWITCH-SPST-SMD-6.2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, SW8 MOMENTARY-SWITCH-SPST-SMD-6.2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, U1 NE555D

Commit message: Updated Lessons 4 and 5
Parts:
- BATT: MOUSER# (none) -> 534-81-8TB; MPN (none) -> 81-8; OC_NEWARK (none) -> unknown
- C1, C2: MOUSER# 791-MT21B104K500CT -> 603-CC805JRX7R9BB104; MPN MT21B104K500CT -> CC805JRX7R9BB104
- Q1: MF INFINION TECHNOLOGIES -> FAIRCHILD SEMICONDUCTOR; MPN BCW66KHE6327HTSA1 -> PN2222ATF
- R1: value 1K -> 3K; MPN CR0805FX-1001ELF -> (none)
- R10, R6: MPN CR0805FX-1001ELF -> (none)
- R2: MPN CR0805FX-1501ELF -> (none)
- R3: MPN CR0805JW-132ELF -> (none)
- R4: MPN CR0805JW-621ELF -> (none)
- R5: MPN CR0805FX-1101ELF -> (none)
- R7: MPN CR0805FX-9100ELF -> (none)
- R8: MPN CR0805JW-391ELF -> (none)
- R9: MPN CR0805FX-6201ELF -> (none)
- SW1, SW2, SW3, SW4, SW5, SW6, SW7, SW8: MOUSER# 653-B3F-1000 -> 693-1301.9317; MPN (none) -> 1301.9317
- U1: MPN TLC555CDR -> (none); OC_NEWARK 24M8296 -> unknown
Changed lines of the file:
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@@
 <attribute name="MF" value=""/>
 <attribute name="MOUSER#" value="595-TLC555CDR"/>
-<attribute name="MPN" value="TLC555CDR"/>
-<attribute name="OC_NEWARK" value="24M8296"/>
+<attribute name="MPN" value=""/>
+<attribute name="OC_NEWARK" value="unknown"/>
 </part>
 <part name="R10" library="rcl" library_urn="urn:adsk.eagle:library:334" deviceset="R-US_" device="R0805" package3d_urn="urn:adsk.eagle:package:23553/2" value="1K">
@@
 <attribute name="MF" value=""/>
 <attribute name="MOUSER#" value="652-CR0805FX-1001ELF"/>
-<attribute name="MPN" value="CR0805FX-1001ELF"/>
+<attribute name="MPN" value=""/>
 <attribute name="OC_NEWARK" value="unknown"/>
 </part>
@@
 <attribute name="MF" value=""/>
 <attribute name="MOUSER#" value="652-CR0805FX-6201ELF"/>
-<attribute name="MPN" value="CR0805FX-6201ELF"/>
+<attribute name="MPN" value=""/>
 <attribute name="OC_NEWARK" value="unknown"/>
 </part>
@@
 <attribute name="MF" value=""/>
 <attribute name="MOUSER#" value="652-CR0805JW-391ELF"/>
-<attribute name="MPN" value="CR0805JW-391ELF"/>
+<attribute name="MPN" value=""/>
 <attribute name="OC_NEWARK" value="unknown"/>
 </part>
@@
 <attribute name="MF" value=""/>
 <attribute name="MOUSER#" value="652-CR0805FX-9100ELF"/>
-<attribute name="MPN" value="CR0805FX-9100ELF"/>
+<attribute name="MPN" value=""/>
 <attribute name="OC_NEWARK" value="unknown"/>
 </part>
@@
 <attribute name="MF" value=""/>
 <attribute name="MOUSER#" value="652-CR0805FX-1001ELF"/>
-<attribute name="MPN" value="CR0805FX-1001ELF"/>
+<attribute name="MPN" value=""/>
 <attribute name="OC_NEWARK" value="unknown"/>
 </part>
@@
 <attribute name="MF" value=""/>
 <attribute name="MOUSER#" value="652-CR0805FX-1101ELF"/>
-<attribute name="MPN" value="CR0805FX-1101ELF"/>
+<attribute name="MPN" value=""/>
 <attribute name="OC_NEWARK" value="unknown"/>
 </part>
@@
 <attribute name="MF" value=""/>
 <attribute name="MOUSER#" value="652-CR0805JW-621ELF"/>
-<attribute name="MPN" value="CR0805JW-621ELF"/>
+<attribute name="MPN" value=""/>
 <attribute name="OC_NEWARK" value="unknown"/>
 </part>
@@
 <attribute name="MF" value=""/>
 <attribute name="MOUSER#" value="652-CR0805JW-132ELF"/>
-<attribute name="MPN" value="CR0805JW-132ELF"/>
+<attribute name="MPN" value=""/>
 <attribute name="OC_NEWARK" value="unknown"/>
 </part>
@@
 <attribute name="MF" value=""/>
 <attribute name="MOUSER#" value="652-CR0805FX-1501ELF"/>
-<attribute name="MPN" value="CR0805FX-1501ELF"/>
+<attribute name="MPN" value=""/>
 <attribute name="OC_NEWARK" value="unknown"/>
 </part>
@@
 </spice>
 <attribute name="MF" value=""/>
-<attribute name="MOUSER#" value="791-MT21B104K500CT"/>
-<attribute name="MPN" value="MT21B104K500CT"/>
+<attribute name="MOUSER#" value="603-CC805JRX7R9BB104"/>
+<attribute name="MPN" value="CC805JRX7R9BB104"/>
 <attribute name="OC_NEWARK" value="unknown"/>
 </part>
 <part name="SW8" library="SparkFun-Switches" library_urn="urn:adsk.eagle:library:535" deviceset="MOMENTARY-SWITCH-SPST" device="-SMD-6.2MM-TALL" package3d_urn="urn:adsk.eagle:package:40172/1" value="MOMENTARY-SWITCH-SPST-SMD-6.2MM-TALL">
 <attribute name="MF" value=""/>
-<attribute name="MOUSER#" value="653-B3F-1000"/>
-<attribute name="MPN" value=""/>
+<attribute name="MOUSER#" value="693-1301.9317"/>
+<attribute name="MPN" value="1301.9317"/>
 <attribute name="OC_NEWARK" value="unknown"/>
 </part>
 <part name="SW7" library="SparkFun-Switches" library_urn="urn:adsk.eagle:library:535" deviceset="MOMENTARY-SWITCH-SPST" device="-SMD-6.2MM-TALL" package3d_urn="urn:adsk.eagle:package:40172/1" value="MOMENTARY-SWITCH-SPST-SMD-6.2MM-TALL">
 <attribute name="MF" value=""/>
-<attribute name="MOUSER#" value="653-B3F-1000"/>
-<attribute name="MPN" value=""/>
+<attribute name="MOUSER#" value="693-1301.9317"/>
+<attribute name="MPN" value="1301.9317"/>
 <attribute name="OC_NEWARK" value="unknown"/>
 </part>
 <part name="SW6" library="SparkFun-Switches" library_urn="urn:adsk.eagle:library:535" deviceset="MOMENTARY-SWITCH-SPST" device="-SMD-6.2MM-TALL" package3d_urn="urn:adsk.eagle:package:40172/1" value="MOMENTARY-SWITCH-SPST-SMD-6.2MM-TALL">
 <attribute name="MF" value=""/>
-<attribute name="MOUSER#" value="653-B3F-1000"/>
-<attribute name="MPN" value=""/>
+<attribute name="MOUSER#" value="693-1301.9317"/>
+<attribute name="MPN" value="1301.9317"/>
 <attribute name="OC_NEWARK" value="unknown"/>
 </part>
 <part name="SW5" library="SparkFun-Switches" library_urn="urn:adsk.eagle:library:535" deviceset="MOMENTARY-SWITCH-SPST" device="-SMD-6.2MM-TALL" package3d_urn="urn:adsk.eagle:package:40172/1" value="MOMENTARY-SWITCH-SPST-SMD-6.2MM-TALL">
 <attribute name="MF" value=""/>
-<attribute name="MOUSER#" value="653-B3F-1000"/>
-<attribute name="MPN" value=""/>
+<attribute name="MOUSER#" value="693-1301.9317"/>
+<attribute name="MPN" value="1301.9317"/>
 <attribute name="OC_NEWARK" value="unknown"/>
 </part>
 <part name="SW4" library="SparkFun-Switches" library_urn="urn:adsk.eagle:library:535" deviceset="MOMENTARY-SWITCH-SPST" device="-SMD-6.2MM-TALL" package3d_urn="urn:adsk.eagle:package:40172/1" value="MOMENTARY-SWITCH-SPST-SMD-6.2MM-TALL">
 <attribute name="MF" value=""/>
-<attribute name="MOUSER#" value="653-B3F-1000"/>
-<attribute name="MPN" value=""/>
+<attribute name="MOUSER#" value="693-1301.9317"/>
+<attribute name="MPN" value="1301.9317"/>
 <attribute name="OC_NEWARK" value="unknown"/>
 </part>
 <part name="SW3" library="SparkFun-Switches" library_urn="urn:adsk.eagle:library:535" deviceset="MOMENTARY-SWITCH-SPST" device="-SMD-6.2MM-TALL" package3d_urn="urn:adsk.eagle:package:40172/1" value="MOMENTARY-SWITCH-SPST-SMD-6.2MM-TALL">
 <attribute name="MF" value=""/>
-<attribute name="MOUSER#" value="653-B3F-1000"/>
-<attribute name="MPN" value=""/>
+<attribute name="MOUSER#" value="693-1301.9317"/>
+<attribute name="MPN" value="1301.9317"/>
 <attribute name="OC_NEWARK" value="unknown"/>
 </part>
 <part name="SW2" library="SparkFun-Switches" library_urn="urn:adsk.eagle:library:535" deviceset="MOMENTARY-SWITCH-SPST" device="-SMD-6.2MM-TALL" package3d_urn="urn:adsk.eagle:package:40172/1" value="MOMENTARY-SWITCH-SPST-SMD-6.2MM-TALL">
 <attribute name="MF" value=""/>
-<attribute name="MOUSER#" value="653-B3F-1000"/>
-<attribute name="MPN" value=""/>
+<attribute name="MOUSER#" value="693-1301.9317"/>
+<attribute name="MPN" value="1301.9317"/>
 <attribute name="OC_NEWARK" value="unknown"/>
 </part>
 <part name="SW1" library="SparkFun-Switches" library_urn="urn:adsk.eagle:library:535" deviceset="MOMENTARY-SWITCH-SPST" device="-SMD-6.2MM-TALL" package3d_urn="urn:adsk.eagle:package:40172/1" value="MOMENTARY-SWITCH-SPST-SMD-6.2MM-TALL">
 <attribute name="MF" value=""/>
-<attribute name="MOUSER#" value="653-B3F-1000"/>
-<attribute name="MPN" value=""/>
+<attribute name="MOUSER#" value="693-1301.9317"/>
+<attribute name="MPN" value="1301.9317"/>
 <attribute name="OC_NEWARK" value="unknown"/>
 </part>
@@
 </spice>
 <attribute name="MF" value=""/>
-<attribute name="MOUSER#" value="791-MT21B104K500CT"/>
-<attribute name="MPN" value="MT21B104K500CT"/>
+<attribute name="MOUSER#" value="603-CC805JRX7R9BB104"/>
+<attribute name="MPN" value="CC805JRX7R9BB104"/>
 <attribute name="OC_NEWARK" value="unknown"/>
 </part>
@@
 <part name="X_3" library="ngspice-simulation" library_urn="urn:adsk.eagle:library:527439" deviceset="GND" device=""/>
 <part name="Q1" library="transistor" library_urn="urn:adsk.eagle:library:402" deviceset="*-NPN-" device="SOT23-BEC" package3d_urn="urn:adsk.eagle:package:28748/2" technology="BCW60" value="BCW66">
-<attribute name="MF" value="INFINION TECHNOLOGIES"/>
+<attribute name="MF" value="FAIRCHILD SEMICONDUCTOR"/>
 <attribute name="MOUSER#" value="726-BCW66KHE6327HTSA"/>
-<attribute name="MPN" value="BCW66KHE6327HTSA1"/>
+<attribute name="MPN" value="PN2222ATF"/>
 <attribute name="OC_NEWARK" value="58K2048"/>
 </part>
 <part name="P+5" library="supply1" library_urn="urn:adsk.eagle:library:371" deviceset="VCC" device=""/>
-<part name="R1" library="rcl" library_urn="urn:adsk.eagle:library:334" deviceset="R-US_" device="R0805" package3d_urn="urn:adsk.eagle:package:23553/2" value="1K">
+<part name="R1" library="rcl" library_urn="urn:adsk.eagle:library:334" deviceset="R-US_" device="R0805" package3d_urn="urn:adsk.eagle:package:23553/2" value="3K">
 <spice>
 <pinmapping spiceprefix="R">
@@
 <attribute name="MF" value=""/>
 <attribute name="MOUSER#" value="652-CR0805FX-1001ELF"/>
-<attribute name="MPN" value="CR0805FX-1001ELF"/>
+<attribute name="MPN" value=""/>
 <attribute name="OC_NEWARK" value="unknown"/>
 </part>
 <part name="X_4" library="ngspice-simulation" library_urn="urn:adsk.eagle:library:527439" deviceset="GND" device=""/>
-<part name="BATT" library="battery" library_urn="urn:adsk.eagle:library:109" deviceset="AB9V" device="" package3d_urn="urn:adsk.eagle:package:4600/1"/>
+<part name="BATT" library="battery" library_urn="urn:adsk.eagle:library:109" deviceset="AB9V" device="" package3d_urn="urn:adsk.eagle:package:4600/1">
+<attribute name="MF" value=""/>
+<attribute name="MOUSER#" value="534-81-8TB"/>
+<attribute name="MPN" value="81-8"/>
+<attribute name="OC_NEWARK" value="unknown"/>
+</part>
 </parts>
 <sheets>
@@
 <attribute name="NAME" x="34.925" y="90.805" size="1.778" layer="95" rot="R90"/>
 <attribute name="VALUE" x="43.18" y="90.805" size="1.778" layer="96" rot="R90"/>
+<attribute name="OC_NEWARK" x="38.1" y="96.52" size="1.778" layer="96" display="off"/>
+<attribute name="MF" x="38.1" y="96.52" size="1.778" layer="96" display="off"/>
+<attribute name="MPN" x="38.1" y="96.52" size="1.778" layer="96" display="off"/>
+<attribute name="MOUSER#" x="38.1" y="96.52" size="1.778" layer="96" rot="R90" display="off"/>
 </instance>
 </instances>
